File: cansat-v3.kicad_sch (KiCad schematic)
At the start: 69 parts, among them J2 USB_C_Receptacle_USB2.0_16P, J3 Micro_SD_Card, Q1 AO3407, SW1 RST, SW2 BOOT, U1 ESP32-S3-WROOM-2, U10 MCP73871, U11 MPU-9250, U2 BME680, U3 TSL25911FN, U4 VEML6075, U5 AP2112K-3.3, U6 INA219BxDCN, U7 NE555D, U8 TPD3E001DRLR, U9 MT3608

Commit message: new desktop first commit
Parts:
- removed BT2: Battery, Connector_JST:JST_XH_B2B-XH-A_1x02_P2.50mm_Vertical, symbol Device:Battery
- removed JP1: SolderJumper_2_Open, Jumper:SolderJumper-2_P1.3mm_Open_TrianglePad1.0x1.5mm, symbol Jumper:SolderJumper_2_Open
- removed Q1: AO3407, Package_TO_SOT_SMD:SOT-23, symbol Transistor_library:Si2323DS
- removed TH1: 10K, Resistor_SMD:R_0603_1608Metric, symbol Device:Thermistor_NTC
- removed U8: TPD3E001DRLR, Package_TO_SOT_SMD:SOT-553, symbol Power_Protection:TPD3E001DRLR
- added C18: 100n, symbol Device:C
- added D6: ~, Diode_SMD:D_SOD-323_HandSoldering, symbol Device:D_TVS
- added FB1: FerriteBead, symbol Device:FerriteBead
- added FB2: 120, symbol Device:FerriteBead
- added R26: 10k, Resistor_SMD:R_1206_3216Metric, symbol Device:R
- added U8: SRV05-4, Package_TO_SOT_SMD:SOT-23-6_Handsoldering, symbol Power_Protection:SRV05-4
- D3: value LED -> Blue
- D4: value LED -> Orange
- D5: value LED -> Green
- J2: footprint Connector_USB:USB_C_Receptacle_G-Switch_GT-USB-7010ASV -> Connector_USB:USB_C_Receptacle_HRO_TYPE-C-31-M-12
- R14: value 1k -> 2k
- R16: value 330 -> 2k
- R17: value 110 -> 2.4k
- R18: value 150 -> 68
- R19: value 150 -> 115
- R20: value 150 -> 100
Connections:
- net +3.3V: now also R16.1; no longer U10.17 (CE)
- net +5V: now also U10.2 (VPCC), FB1.2, U8.5 (VP); no longer R16.1
- net +BATT: now also U10.16 (V_{BAT_SENSE})
- net GND: now also R17.2, U10.3 (SEL), C18.2, D6.1 (A1), FB2.1, R26.2, U8.2 (VN); no longer J2.A1 (GND), J2.A12 (GND), J2.B1 (GND), J2.B12 (GND), R17.1
- net USB_D+: now also J2.A6 (D+), J2.B6 (D+), U8.6 (IO4); no longer J2.A7 (D-), J2.B7 (D-)
- net USB_D-: now also J2.A7 (D-), J2.B7 (D-), U8.1 (IO1); no longer J2.A6 (D+), J2.B6 (D+)
- net VBUS: now also FB1.1
- net Earth: now reaches J2.S1 (SHIELD)
- net Earth: now also J2.A1 (GND), J2.A12 (GND), J2.B1 (GND), J2.B12 (GND), C18.1, D6.2 (A2), FB2.2
- net at R19.2: now also U10.6 (~{PG}); no longer U10.8 (STAT1/~{LBO})
- net at U10.5 (THERM): now also R26.1
- net at R18.2: now also U10.7 (STAT2); no longer U10.6 (~{PG})
- net at R20.2: now also U10.8 (STAT1/~{LBO}); no longer U10.7 (STAT2)
- new net: R16.2, R17.1, U10.17 (CE)
Other:
- note removed: "Charge -> 1000mA"
- note removed: "Charge -> 500mA"
- moved on the sheet: BT1, C10, C11, C12, C13, C14, C15, C16, C17, C6, C7, C8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

Commit message: autopush test
Parts:
- added R27, R28: 4.7k, Resistor_SMD:R_0603_1608Metric, symbol Device:R
- added U12: SCD40-D-R2, Sensor:Sensirion_SCD4x-1EP_10.1x10.1mm_P1.25mm_EP4.8x4.8mm, symbol Sensor_Gas:SCD40-D-R2
Connections:
- net +3.3V: now also R27.1, R28.1, U12.19 (VDD), U12.7 (VDD)
- new net: U12.20 (GND), U12.21 (GND), U12.6 (GND)
- new net SCD40_SCL: R28.2, U12.9 (SCL)
- new net SCD40_SDA: R27.2, U12.10 (SDA)
Other:
- moved on the sheet: J3

Commit message: Sensor development
Parts:
- removed SW1: RST, Button_Switch_SMD:SW_MEC_5GSH9, symbol Switch:SW_MEC_5E
- removed SW2: BOOT, Button_Switch_SMD:SW_MEC_5GSH9, symbol Switch:SW_MEC_5E
- added C19: 0.1u, Capacitor_SMD:C_0603_1608Metric, symbol Device:C
- added C20: 1u, Capacitor_SMD:C_0603_1608Metric, symbol Device:C
- added C21: 0.12u, Capacitor_SMD:C_0603_1608Metric, symbol Device:C
- added R29: 10k, Resistor_SMD:R_0603_1608Metric, symbol Device:R
- added R30, R31: 4.7k, Resistor_SMD:R_0603_1608Metric, symbol Device:R
- added SW1, SW3: KMR223G, Button_Switch_SMD:SW_Push_1P1T-SH_NO_CK_KMR2xxG, symbol Switch:SW_Push_Shielded
- added U13: BNO055, Package_LGA:LGA-28_5.2x3.8mm_P0.5mm, symbol Sensor_Motion:BNO055
- added U14: AS7331-AQFM, AS7331-AQFM:PQFN50P365X260X119-16N, symbol AS7331-AQFM:AS7331-AQFM
- C14, C17, C8, D1, L1, R12, R2, R21, R22, R23, R5, U11, U4, U7, U9: now left out of the parts list
- R27, R28: value 4.7k -> 10k
Connections:
- net +3.3V: now also C19.1, R29.1, R30.2, R31.2, U13.3 (VDD)
- net GND: now also U12.20 (GND), U12.21 (GND), U12.6 (GND), C19.2, C20.1, C21.1, SW1.2, SW1.SH (B), SW3.1, SW3.SH (B), U13.17 (COM3), U13.18 (COM2), U13.2 (GND), U13.25 (GNDIO), U13.5 (PS1), U13.6 (PS0)
- net RST: now also SW3.2
- net Boot: no longer names the net of C5.2, U1.27 (IO0)
- net Boot: now also SW1.1
- new net: C21.2, U13.28 (VDDIO)
- new net: R29.2, U13.4 (~{BOOT_LOAD_PIN})
- new net: C20.2, U13.9 (CAP)
- new net: U14.1 (VSSA), U14.15 (VSSA), U14.16 (VSSA), U14.2 (VSSA), U14.5 (VSSA), U14.6 (VSSA)
- new net BNO055_RST: U13.11 (~{RESET})
- new net BNO055_SCL: R30.1, U13.19 (COM1)
- new net BNO055_SDA: R31.1, U13.20 (COM0)
- no-connect marks 6 -> 10
Other:
- note added: "0x28"
- moved on the sheet: C5, C8, R2, R3, R5, R6, R8, U11, U3, U4

Commit message: Power subsystem finished, Sensors continued
Parts:
- removed U5: AP2112K-3.3, Package_TO_SOT_SMD:SOT-23-5, symbol Regulator_Linear:AP2112K-3.3
- added C22, C23, C24: 0.1u, Capacitor_SMD:C_0603_1608Metric, symbol Device:C
- added C25, C26: 22n, Capacitor_SMD:C_0603_1608Metric, symbol Device:C
- added D7: LED, LED_SMD:LED_1206_3216Metric_Pad1.42x1.75mm_HandSolder, symbol Device:LED
- added JP2: SolderJumper_2_Bridged, Jumper:SolderJumper-2_P1.3mm_Bridged2Bar_RoundedPad1.0x1.5mm, symbol Jumper:SolderJumper_2_Bridged
- added R32, R36: 10k, symbol Device:R_Small
- added R33: 3.3M, symbol Device:R
- added R34, R35: 820, symbol Device:R
- added R37: 66.5, Resistor_SMD:R_1206_3216Metric, symbol Device:R
- added SW2: PWR, symbol Switch:SW_SPDT
- added U15: Digital PS, RT9193-33GB:SOT94P279X129-5N, symbol RT9193-33GB:RT9193-33GB
- added U5: Analog PS, RT9193-33GB:SOT94P279X129-5N, symbol RT9193-33GB:RT9193-33GB
- C11: value 1u -> 0.1u
- C9: value 1u -> 470u
Connections:
- net +3.3V: now also U14.10 (VDDD), C22.1, C24.2, R34.2, R35.2, U15.5 (VOUT); no longer C11.1
- net +BATT: now also SW2.1 (A)
- net GND: now also C11.1, U14.11 (VSSD), C22.2, C24.1, C25.1, C26.1, D7.1 (K), JP2.1 (A), R32.2, R36.2, U15.2 (GND), U5.2 (GND); no longer C11.2, C9.2
- net at C9.1, D89.1 (K): now also C9.2, U15.1 (VIN), U5.1 (VIN)
- net VSSA: now reaches U14.1 (VSSA), U14.15 (VSSA), U14.16 (VSSA), U14.2 (VSSA), U14.5 (VSSA), U14.6 (VSSA)
- net VSSA: now also U14.14 (A0), U14.7 (A1), C23.2, JP2.2 (B), R33.2
- net AS7331_SDA: now reaches U14.12 (SDA)
- net AS7331_SDA: now also R34.1
- net AS7331_SCL: now reaches U14.13 (SCL)
- net AS7331_SCL: now also R35.1
- net VDDA: now reaches U14.3 (VDDA)
- net VDDA: now also C11.2, C23.1, R37.1, U5.5 (VOUT)
- net at U14.4 (REXT): now also R33.1
- new net: C26.2, U15.4 (BP)
- new net: D7.2 (A), R37.2
- new net: C25.2, U5.4 (BP)
- new net PWR_EN: R32.1, R36.1, SW2.2 (B), U15.3 (EN), U5.3 (EN)
- no-connect marks 10 -> 13
Other:
- note added: "Components on same side"
- note added: "MCU"
- note added: "Power"
- note added: "Sensors"
- note removed: "ENS160"
- moved on the sheet: C1, C14, C17, C18, C19, C2, C20, C21, C3, C4, C5, C6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

Commit message: Started layout
Parts:
- removed SW1, SW3: KMR223G, Button_Switch_SMD:SW_Push_1P1T-SH_NO_CK_KMR2xxG, symbol Switch:SW_Push_Shielded
- removed U12: SCD40-D-R2, Sensor:Sensirion_SCD4x-1EP_10.1x10.1mm_P1.25mm_EP4.8x4.8mm, symbol Sensor_Gas:SCD40-D-R2
- added C27, C28: 0.1u, Capacitor_SMD:C_0603_1608Metric, symbol Device:C
- added J1: Conn_01x04_Socket, Connector_JST:JST_XH_B4B-XH-A_1x04_P2.50mm_Vertical, symbol Connector:Conn_01x04_Socket
- added J4: Conn_01x02_Socket, Connector_JST:JST_XH_B2B-XH-A_1x02_P2.50mm_Vertical, symbol Connector:Conn_01x02_Socket
- added J5: Conn_01x05_Socket, Connector_JST:JST_XH_B5B-XH-A_1x05_P2.50mm_Vertical, symbol Connector:Conn_01x05_Socket
- added SW1, SW3: SW_Push, Button_Switch_SMD:Panasonic_EVQPUJ_EVQPUA, symbol Switch:SW_Push
- added U12: SCD40-D-R2, Sensor:Sensirion_SCD4x-1EP_10.1x10.1mm_P1.25mm_EP4.8x4.8mm, symbol custom:SCD40-D-R2
- BT1: footprint Connector_AMASS:AMASS_XT60-F_1x02_P7.20mm_Vertical -> Connector_JST:JST_XH_B2B-XH-A_1x02_P2.50mm_Vertical
- C18: footprint (none) -> Capacitor_SMD:C_0603_1608Metric
- FB1: value FerriteBead -> LI0603G121R-10; footprint (none) -> Inductor_SMD:L_0603_1608Metric
- FB2: value 120 -> LI0603G121R-10; footprint (none) -> Inductor_SMD:L_0603_1608Metric
- R13, R14, R15, R16, R17, R18, R19, R20, R24, R25, R26, R37: footprint Resistor_SMD:R_1206_3216Metric -> Resistor_SMD:R_0603_1608Metric
- R32, R33, R34, R35, R36: footprint (none) -> Resistor_SMD:R_0603_1608Metric
- SW2: footprint (none) -> Button_Switch_THT:SW_E-Switch_EG1224_SPDT_Angled
Connections:
- net +3.3V: now also J1.1 (Pin_1), J5.1 (Pin_1), U12.19 (VDD), U12.7 (VDD)
- net GND: now also C27.2, C28.1, J1.2 (Pin_2), J5.4 (Pin_4), SW1.2, SW3.1, U12.20 (GND), U12.21 (GND), U12.6 (GND)
- net RST: now also SW3.2
- net SCD40_SCL: now also U12.9 (SCL)
- net SCD40_SDA: now also U12.10 (SDA)
- net at C5.2, U1.27 (IO0): now also SW1.1
- net at C9.1, C9.2, D89.1 (K)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: now also C27.1, C28.2
- new net: U12.1 (NC), U12.11 (NC), U12.12 (NC), U12.13 (NC), U12.14 (NC), U12.15 (NC), U12.16 (NC), U12.17 (NC), U12.18 (NC), U12.2 (NC), U12.3 (NC), U12.4 (NC), U12.5 (NC), U12.8 (NC)
- new net COMPASS_SCL: J4.2 (Pin_2)
- new net COMPASS_SDA: J4.1 (Pin_1)
- new net GPS_RX: J1.3 (Pin_3)
- new net GPS_TX: J1.4 (Pin_4)
- new net LoRa_RST: J5.5 (Pin_5)
- new net LoRa_RX: J5.3 (Pin_3)
- new net LoRa_TX: J5.2 (Pin_2)
Other:
- note added: "pin 1 of the lora cs1 isn't used"
- moved on the sheet: BT1

Commit message: Component placement finished, started routing
Parts:
- added H1, H2, H3, H4: MountingHole_Pad, MountingHole:MountingHole_4.3mm_M4_Pad, symbol Mechanical:MountingHole_Pad
Connections:
- net AS7331_SCL: now also U1.33 (MTDO/IO40)
- net AS7331_SDA: now also U1.34 (MTDI/IO41)
- net BME680_SCL: now also U1.15 (IO3)
- net BME680_SDA: now also U1.16 (IO46)
- net BNO055_RST: now also U1.23 (IO21)
- net BNO055_SCL: now also U1.31 (IO38)
- net BNO055_SDA: now also U1.26 (IO45)
- net COMPASS_SCL: now also U1.17 (IO9)
- net COMPASS_SDA: now also U1.18 (IO10)
- net GND: now also H1.1, H2.1, H3.1, H4.1
- net GPS_RX: now also U1.21 (IO13)
- net GPS_TX: now also U1.22 (IO14)
- net INA219_SCL: now also U1.20 (IO12)
- net INA219_SDA: now also U1.19 (IO11)
- net LoRa_RST: now also U1.32 (MTCK/IO39)
- net LoRa_RX: now also U1.36 (RXD0/IO44)
- net LoRa_TX: now also U1.37 (TXD0/IO43)
- net SCD40_SCL: now also U1.10 (IO17)
- net SCD40_SDA: now also U1.11 (IO18)
- net SD_CLK: now also U1.6 (IO6)
- net SD_CS: now also U1.4 (IO4)
- net SD_MISO: now also U1.7 (IO7)
- net SD_MOSI: now also U1.5 (IO5)
- net TSL2591_SCL: now also U1.9 (IO16)
- net TSL2591_SDA: now also U1.8 (IO15)
- net USB_D+: now also U1.14 (USB_D+/IO20), U8.1 (IO1); no longer U8.6 (IO4)
- net USB_D-: now also U1.13 (USB_D-/IO19), U8.6 (IO4); no longer U8.1 (IO1)
- no-connect marks 13 -> 15
